File: Thiết kế PCB/Smart_Garden.kicad_sch (KiCad schematic)
At the start: 30 parts, among them J1 Conn_02x03_Top_Bottom, J2 Conn_01x04_Socket, J3 Conn_01x03_Socket, J4 Conn_01x04_Socket, J5 USB_B, J6 Conn_01x04_Socket, SW1 SW_Push, U1 DHT11, U2 ATmega328P-P, Y1 16MHz

Commit message: update name
Other:
- company: (none) -> Author : Vương Toàn Hội - Phạm Ngọc Ánh
- title: (none) -> Smart Garden
Changed lines of the file:
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@@
 	(generator_version "8.0")
 	(paper "A4")
+	(title_block
+		(title "Smart Garden")
+		(date "2025-05-12")
+		(rev "1.1")
+		(company "Author : Vương Toàn Hội - Phạm Ngọc Ánh")
+	)
 	(junction
 		(at 60.96 35.56)
